Commit message: Mejora de simulación: Optimización 3D, control Xbox y cámara 30fps

File: src/mi_proyecto_sim/urdf/carrito_con_aruco.urdf.xacro (robot description, xacro)
@@ -28,7 +28,8 @@
         <parent link="base_link"/>
         <child link="techo_aruco_link"/>
-        <origin xyz="0 0 0.18" rpy="0 0 0"/>
+        <origin xyz="0 0 0.19" rpy="0 0 0"/>
     </joint>
     <gazebo>
+        <!--
         <plugin filename="libignition-gazebo-mecanum-drive-system.so" name="ignition::gazebo::systems::MecanumDrive">
             <front_left_joint>front_left_wheel_joint</front_left_joint>
@@ -41,4 +42,5 @@
             <topic>/cmd_vel</topic>
         </plugin>
+        -->
         <plugin filename="libignition-gazebo-velocity-control-system.so" name="ignition::gazebo::systems::VelocityControl">
             <topic>/cmd_vel</topic>

Commit message: feat: Navegación autónoma con fusión continua ArUco+Odometría
- Activar plugin MecanumDrive para odometría física real
- Implementar fusión continua (90% odom / 10% ArUco) con filtro pasa-baja
- Lectura directa de /odom por tópico (bypass de TF para robustez en Gazebo Sim)
- Fallback a ArUco crudo cuando la odometría no está disponible al arrancar
- Evasión reactiva con umbral dinámico (35cm frente, 15cm lados)
- Suavizado de velocidad con filtro pasa-baja
- Puente ros_gz_bridge para /odom y /tf desde Gazebo
- Añadir filtro_lidar.py (recorte de campo de visión a 110°)
- Actualizar README con arquitectura del sistema

File: src/mi_proyecto_sim/urdf/carrito_con_aruco.urdf.xacro (robot description, xacro)
@@ -1,14 +1,15 @@
 <?xml version="1.0"?>
 <robot name="rosmaster_x3_aruco" xmlns:xacro="http://www.ros.org/wiki/xacro">
-    <xacro:include filename="$(find yahboom_rosmaster_description)/urdf/robots/rosmaster_x3.urdf.xacro" />
+    <xacro:include
+        filename="$(find yahboom_rosmaster_description)/urdf/robots/rosmaster_x3.urdf.xacro" />
     <link name="techo_aruco_link">
         <visual>
             <geometry>
-                <box size="0.15 0.15 0.001"/>
+                <box size="0.15 0.15 0.001" />
             </geometry>
         </visual>
         <inertial>
-            <mass value="0.1"/>
-            <inertia ixx="0.001" ixy="0" ixz="0" iyy="0.001" iyz="0" izz="0.001"/>
+            <mass value="0.1" />
+            <inertia ixx="0.001" ixy="0" ixz="0" iyy="0.001" iyz="0" izz="0.001" />
         </inertial>
     </link>
@@ -26,11 +27,11 @@
     </gazebo>
     <joint name="aruco_base_joint" type="fixed">
-        <parent link="base_link"/>
-        <child link="techo_aruco_link"/>
-        <origin xyz="0 0 0.19" rpy="0 0 0"/>
+        <parent link="base_link" />
+        <child link="techo_aruco_link" />
+        <origin xyz="0 0 0.19" rpy="0 0 0" />
     </joint>
     <gazebo>
-        <!--
-        <plugin filename="libignition-gazebo-mecanum-drive-system.so" name="ignition::gazebo::systems::MecanumDrive">
+        <plugin filename="libignition-gazebo-mecanum-drive-system.so"
+            name="ignition::gazebo::systems::MecanumDrive">
             <front_left_joint>front_left_wheel_joint</front_left_joint>
             <front_right_joint>front_right_wheel_joint</front_right_joint>
@@ -40,10 +41,16 @@
             <wheelbase>0.16</wheelbase>
             <wheel_radius>0.0325</wheel_radius>
+            <odom_frame>odom</odom_frame>
+            <robot_base_frame>base_footprint</robot_base_frame>
+            <publish_odom>true</publish_odom>
+            <publish_odom_tf>true</publish_odom_tf>
+            <topic>/cmd_vel</topic>
+        </plugin>
+        <!-- (VelocityControl comentado para usar MecanumDrive con fisica real)
+        <plugin filename="libignition-gazebo-velocity-control-system.so"
+        name="ignition::gazebo::systems::VelocityControl">
             <topic>/cmd_vel</topic>
         </plugin>
         -->
-        <plugin filename="libignition-gazebo-velocity-control-system.so" name="ignition::gazebo::systems::VelocityControl">
-            <topic>/cmd_vel</topic>
-        </plugin>
     </gazebo>
 </robot>

Commit message: Optimización de escape en esquinas, escala de mapa 1:1 y rotación pura inicial

File: src/mi_proyecto_sim/urdf/carrito_con_aruco.urdf.xacro (robot description, xacro)
@@ -6,5 +6,5 @@
         <visual>
             <geometry>
-                <box size="0.15 0.15 0.001" />
+                <box size="0.18 0.18 0.001" />
             </geometry>
         </visual>

Commit message: feat: optimizacion de mision, control de trayectoria y calibracion de ArUcos
- Control de trayectoria: Reducido el umbral de llegada a meta a 5 cm (pos_threshold = 0.05) para mayor precision.
- Mision dron: Implementada calibracion dinamica con offsets de guiñada (yaw) personalizados por ID de marcador ArUco (ARUCO_YAW_OFFSETS). Corregida la comprobacion de estado DONE ante interrupciones.
- URDF: Añadida la etiqueta de colision (<collision>) al marcador ArUco en el carrito_con_aruco.urdf.xacro.
- Launch: Creado el launch file 'control_con_obstaculos.launch.py' para spawnear obstaculos variables de forma diferida antes de iniciar el control.
- Mapas: Guardados y actualizados los nuevos mapas de ocupacion generados (occupancy_map, mapa_mision y ubicaciones de ArUcos).

File: src/mi_proyecto_sim/urdf/carrito_con_aruco.urdf.xacro (robot description, xacro)
@@ -9,4 +9,9 @@
             </geometry>
         </visual>
+        <collision>
+            <geometry>
+                <box size="0.18 0.18 0.001" />
+            </geometry>
+        </collision>
         <inertial>
             <mass value="0.1" />
