Commit message: feat(sim): control pid sim-to-real y optimizacion de llantas mecanum
- Implementacion de Mcnamu_driver_PID_sim.py con mapeo lineal PWM a Esfuerzo (Nm) para usar ganancias reales de control en simulacion.
- Modificaciones en launchs (simulacion, solo_carrito, test_pid) para cargar el driver PID y ros2_control.
- Ajuste del centro de masa del Rosmaster a (0,0) para eliminar el drift de yaw en strafe.
- Optimizacion del URDF de llantas mecanum reduciendo la cantidad de rodillos de 12 a 6 por rueda para mejorar drasticamente el RTF en Ignition Gazebo.
- Ajuste en laberinto.sdf para restaurar controles GUI y visualizacion de RTF.

File: src/yahboom_rosmaster/yahboom_rosmaster_description/urdf/mech/mecanum_wheel.urdf.xacro (robot description, xacro)
@@ -4,7 +4,43 @@
   <xacro:property name="wheel_separation" value="0.169" />
   <xacro:property name="wheel_width" value="0.03040" />
-  <xacro:property name="wheel_mass" value="9.1" />
+  <xacro:property name="wheel_mass" value="0.15" />
+  <xacro:property name="roller_mass" value="0.02" />
+  <xacro:property name="roller_radius" value="0.0065" />
   <xacro:property name="wheel_xoff" value="0.08" />
   <xacro:property name="wheel_yoff" value="-0.01" />
+  <xacro:macro name="mecanum_roller" params="prefix side index theta alpha">
+    <link name="${prefix}${side}_roller_${index}_link">
+      <collision>
+        <origin xyz="0 0 0" rpy="0 0 0"/>
+        <geometry>
+          <sphere radius="${roller_radius}"/>
+        </geometry>
+        <max_contacts>2</max_contacts>
+      </collision>
+      <inertial>
+        <mass value="${roller_mass}"/>
+        <inertia ixx="${2.0/5.0 * roller_mass * roller_radius * roller_radius}" ixy="0" ixz="0"
+                 iyy="${2.0/5.0 * roller_mass * roller_radius * roller_radius}" iyz="0"
+                 izz="${2.0/5.0 * roller_mass * roller_radius * roller_radius}"/>
+      </inertial>
+    </link>
+    <joint name="${prefix}${side}_roller_${index}_joint" type="continuous">
+      <parent link="${prefix}${side}_wheel_link"/>
+      <child link="${prefix}${side}_roller_${index}_link"/>
+      <axis xyz="${sin(alpha)} ${cos(alpha)} 0"/>
+      <origin xyz="${(wheel_radius - roller_radius)*sin(theta)} 0 ${(wheel_radius - roller_radius)*cos(theta)}" rpy="0 ${theta} 0"/>
+      <dynamics damping="0.001" friction="0.001"/>
+    </joint>
+    <gazebo reference="${prefix}${side}_roller_${index}_link">
+      <mu1>1.0</mu1>
+      <mu2>1.0</mu2>
+      <kp>10000.0</kp>
+      <kd>10.0</kd>
+      <minDepth>0.001</minDepth>
+      <maxVel>1.0</maxVel>
+      <self_collide>false</self_collide>
+      <max_contacts>2</max_contacts>
+    </gazebo>
+  </xacro:macro>
   <xacro:macro name="mecanum_wheel" params="prefix side x_reflect y_reflect">
     <link name="${prefix}${side}_wheel_link">
@@ -18,10 +54,4 @@
         </material>
       </visual>
-      <collision>
-        <origin xyz="0 0 0" rpy="0 0 0"/>
-        <geometry>
-          <sphere radius="${wheel_radius}"/>
-        </geometry>
-      </collision>
       <inertial>
         <origin xyz="0 0 0" rpy="0 0 0"/>
@@ -38,14 +68,7 @@
       <child link="${prefix}${side}_wheel_link"/>
       <origin xyz="${x_reflect*wheel_xoff} ${y_reflect*(wheel_separation/2+wheel_yoff)} ${-wheel_radius}" rpy="0 0 0"/>
+      <dynamics damping="0.2" friction="0.1"/>
     </joint>
     <gazebo reference="${prefix}${side}_wheel_link">
-      <surface>
-        <friction>
-          <ode>
-              <mu>1.0</mu>
-              <mu2>0.5</mu2>
-          </ode>
-        </friction>
-      </surface>
       <visual>
           <material>
@@ -54,5 +77,13 @@
           </material>
       </visual>
+      <self_collide>false</self_collide>
     </gazebo>
+    <xacro:property name="alpha" value="${(x_reflect * y_reflect) * (pi / 4)}" />
+    <xacro:mecanum_roller prefix="${prefix}" side="${side}" index="0" theta="0.0" alpha="${alpha}" />
+    <xacro:mecanum_roller prefix="${prefix}" side="${side}" index="1" theta="${pi/3}" alpha="${alpha}" />
+    <xacro:mecanum_roller prefix="${prefix}" side="${side}" index="2" theta="${2*pi/3}" alpha="${alpha}" />
+    <xacro:mecanum_roller prefix="${prefix}" side="${side}" index="3" theta="${3*pi/3}" alpha="${alpha}" />
+    <xacro:mecanum_roller prefix="${prefix}" side="${side}" index="4" theta="${4*pi/3}" alpha="${alpha}" />
+    <xacro:mecanum_roller prefix="${prefix}" side="${side}" index="5" theta="${5*pi/3}" alpha="${alpha}" />
   </xacro:macro>
 </robot>

File: src/yahboom_rosmaster/yahboom_rosmaster_description/urdf/mech/rosmaster_x3_base.urdf.xacro (robot description, xacro)
@@ -31,5 +31,6 @@
     </collision>
     <inertial>
-        <origin xyz="${base_x_offset} 0 ${base_size_z/2 + wheel_radius/4}" rpy="0 0 0"/>
+        <!-- SIM-TO-REAL FIX: Centramos el CoM en X=0 y Y=0 para evitar que el robot rote al hacer strafe -->
+        <origin xyz="0 0 ${base_size_z/2 + wheel_radius/4}" rpy="0 0 0"/>
         <mass value="${base_mass}"/>
         <inertia
