Commit message: feat(sim-to-real): control de parqueo visual_servo omnidireccional y fix de hardware driver
- control_trayectoria: Completado el algoritmo de visual_servo usando control mecanum omnidireccional. Ahora la rotacion angular centra el marker, cmd.linear.y corrige la asimetria lateral para perpendicularidad, y cmd.linear.x maneja la distancia (area). Ademas, se corrigio el terminal_approach_mode convirtiendolo en go-to-point omnidireccional simultaneo para evitar atascos de rotacion.
- rosmaster_x3_base: Revertido el CoM al centro de masa fisico original con base_x_offset.
- Mcnamu_driver_PID (real): Aplicado fix critico de Sim-To-Real. El feedforward ahora incorpora la banda muerta (u_base = copysign(deadband, w_ref)) de forma que la senal de velocidad minima para romper inercia se aplique de inmediato, previniendo que el robot real se quede congelado.

File: src/yahboom_rosmaster/yahboom_rosmaster_description/urdf/mech/rosmaster_x3_base.urdf.xacro (robot description, xacro)
@@ -31,6 +31,5 @@
     </collision>
     <inertial>
-        <!-- SIM-TO-REAL FIX: Centramos el CoM en X=0 y Y=0 para evitar que el robot rote al hacer strafe -->
-        <origin xyz="0 0 ${base_size_z/2 + wheel_radius/4}" rpy="0 0 0"/>
+        <origin xyz="${base_x_offset} 0 ${base_size_z/2 + wheel_radius/4}" rpy="0 0 0"/>
         <mass value="${base_mass}"/>
         <inertia
