Commit message: Mejora de visual servoing: integracion de solvePnP para asimetria 3D y ajuste de distancia de estacionamiento

File: src/mi_proyecto_sim/urdf/jetauto/jetauto_sensors.urdf.xacro (robot description, xacro)
@@ -122,5 +122,5 @@
     </link>
     <joint name="${prefix}cam_1_joint" type="fixed">
-      <origin xyz="0.0288581470059471 0 0.202093286991617" rpy="0 0 0"/>
+      <origin xyz="0.0288581470059471 0 0.202093286991617" rpy="0 0.261 0"/>
       <parent link="${prefix}base_link"/>
       <child  link="${prefix}cam_1_link"/>

Commit message: Sim: MS200 sobre soporte Legera + lidar igualado al real + sin recorte de FOV
Lleva el lidar de la simulacion a paridad con el robot real (Orbbec MS200
montado sobre el soporte impreso Legera) y elimina el filtro artificial de FOV.

URDF / modelo:
- jetauto_soporte.urdf.xacro (nuevo): soporte Legera + ArUco 3D (ID 4) + cuerpo
  MS200 (malla CAD re-teselada con gmsh, sin bracket) + lidar_frame. SIN colision
  en support_link/ms200_link para que el gpu_lidar no se vea a si mismo -> /scan
  crudo limpio en 360.
- jetauto_sim: wiring use_soporte (default true); con soporte, el ArUco 3D
  reemplaza al plano.
- jetauto_sensors: con soporte, el MS200 da /scan (lidar_frame) y el A1 queda como
  secundario en /scan_a1 (presente, sin usar). El A1 "unless soporte" actualizado a
  7.65 Hz/360 pts (su spec real medida).

Lidar gz = specs reales del MS200 (driver oradar): 15 Hz, ~300 pts/scan, 360 deg,
rango 0.03-12 m, ruido sigma 0.0043 m (caracterizacion estatica en piso).

Sin filtro de FOV:
- filtro_lidar: parametro half_fov_deg (default 180 = 360 completo); conserva solo
  el self_clearance de auto-oclusion. (El robot real lo sigue usando.)
- control/slam/amcl: scan_topic parametrizable (default /scan); las launches reales
  pasan /scan_filtered para conservar el filtro en hardware.
- filtro_lidar quitado de las launches de sim; configs mapper/amcl -> /scan.

File: src/mi_proyecto_sim/urdf/jetauto/jetauto_sensors.urdf.xacro (robot description, xacro)
@@ -13,4 +13,7 @@
   <xacro:macro name="jetauto_sensors" params="prefix">
     <!-- ===================== LiDAR (RPLIDAR A1) ===================== -->
+    <!-- Solo cuando NO se usa el soporte 3D. Con use_soporte:=true, el MS200 sobre el
+         soporte provee /scan en el frame lidar_frame (ver jetauto_soporte.urdf.xacro). -->
+    <xacro:unless value="$(arg use_soporte)">
     <link name="${prefix}lidar_link">
       <inertial>
@@ -41,5 +44,6 @@
       <sensor name="${prefix}lidar_a1" type="gpu_lidar">
         <topic>scan</topic>
-        <update_rate>10</update_rate>
+        <!-- sim-to-real: lidar real medido a ~7.65 Hz (scan_time 0.131 s), 360 pts (1 deg) -->
+        <update_rate>7.65</update_rate>
         <always_on>1</always_on>
         <visualize>false</visualize>
@@ -48,5 +52,5 @@
           <scan>
             <horizontal>
-              <samples>720</samples>
+              <samples>360</samples>   <!-- 1 grado/punto, como el lidar real (angle_increment 0.0175) -->
               <resolution>1</resolution>
               <min_angle>-3.14159265</min_angle>
@@ -73,4 +77,57 @@
       </sensor>
     </gazebo>
+    </xacro:unless>
+    <!-- ===== RPLIDAR A1 SECUNDARIO (cuando hay soporte): mismo pod en su posicion original,
+         pero en frame lidar_a1_frame y publicando en /scan_a1. Presente pero NO lo usa nav
+         (el MS200 es /scan). Para activarlo en nav, remapea /scan_a1 -> /scan donde toque. -->
+    <xacro:if value="$(arg use_soporte)">
+    <link name="${prefix}lidar_link">
+      <inertial>
+        <origin xyz="-0.0157049024536227 0.000340793431659825 -0.0214732100882973" rpy="0 0 0"/>
+        <mass value="0.0522535578752524"/>
+        <inertia ixx="1.4542908499666E-05" ixy="4.8193721668021E-08" ixz="2.30575406031324E-07"
+                 iyy="1.85618648837978E-05" iyz="-1.29750110413905E-08" izz="3.10574357987674E-05"/>
+      </inertial>
+      <visual>
+        <origin xyz="0 0 0" rpy="0 0 0"/>
+        <geometry><mesh filename="${mesh_dir}/lidar_link.stl"/></geometry>
+        <material name="lidar_black"><color rgba="0.1 0.1 0.1 1.0"/></material>
+      </visual>
+    </link>
+    <joint name="${prefix}lidar_joint" type="fixed">
+      <origin xyz="0.0959394346777203 -1.03974386779226E-05 0.128396206697751" rpy="0 0 0"/>
+      <parent link="${prefix}base_link"/>
+      <child  link="${prefix}lidar_link"/>
+    </joint>
+    <link name="${prefix}lidar_a1_frame"/>
+    <joint name="${prefix}lidar_a1_frame_joint" type="fixed">
+      <origin xyz="0 0 0" rpy="0 0 ${M_PI}"/>
+      <parent link="${prefix}lidar_link"/>
+      <child  link="${prefix}lidar_a1_frame"/>
+    </joint>
+    <gazebo reference="${prefix}lidar_a1_frame">
+      <sensor name="${prefix}lidar_a1" type="gpu_lidar">
+        <topic>scan_a1</topic>
+        <update_rate>7.65</update_rate>
+        <always_on>1</always_on>
+        <visualize>false</visualize>
+        <gz_frame_id>${prefix}lidar_a1_frame</gz_frame_id>
+        <lidar>
+          <scan>
+            <horizontal>
+              <samples>360</samples><resolution>1</resolution>
+              <min_angle>-3.14159265</min_angle><max_angle>3.14159265</max_angle>
+            </horizontal>
+            <vertical>
+              <samples>1</samples><resolution>1</resolution>
+              <min_angle>0</min_angle><max_angle>0</max_angle>
+            </vertical>
+          </scan>
+          <range><min>0.15</min><max>12.0</max><resolution>0.013</resolution></range>
+          <noise><type>gaussian</type><mean>0.0</mean><stddev>0.01</stddev></noise>
+        </lidar>
+      </sensor>
+    </gazebo>
+    </xacro:if>
     <!-- ===================== IMU (MPU-6050) ===================== -->
     <link name="${prefix}imu_link">

File: src/mi_proyecto_sim/urdf/jetauto/jetauto_sim.urdf.xacro (robot description, xacro)
@@ -18,8 +18,12 @@
   <xacro:arg name="prefix"     default=""/>
   <xacro:arg name="use_aruco"  default="true"/>
+  <!-- use_soporte=true (DEFAULT): soporte 3D (Legera) + ArUco 3D + MS200 (/scan, lidar_frame) +
+       A1 secundario (/scan_a1). use_soporte=false: config original (A1 en /scan, ArUco plano). -->
+  <xacro:arg name="use_soporte" default="true"/>
   <xacro:include filename="$(find mi_proyecto_sim)/urdf/jetauto/jetauto_base.urdf.xacro"/>
   <xacro:include filename="$(find mi_proyecto_sim)/urdf/jetauto/jetauto_mecanum_wheel.urdf.xacro"/>
   <xacro:include filename="$(find mi_proyecto_sim)/urdf/jetauto/jetauto_sensors.urdf.xacro"/>
   <xacro:include filename="$(find mi_proyecto_sim)/urdf/jetauto/jetauto_control.urdf.xacro"/>
+  <xacro:include filename="$(find mi_proyecto_sim)/urdf/jetauto/jetauto_soporte.urdf.xacro"/>
   <!-- chassis + decorative shells -->
   <xacro:jetauto_base prefix="$(arg prefix)"/>
@@ -33,6 +37,7 @@
   <!-- velocity ros2_control + ign_ros2_control -->
   <xacro:jetauto_control prefix="$(arg prefix)"/>
-  <!-- ArUco marker on the roof (used by the drone/mission to localize the carrito).
-       Same as the original carrito_con_aruco; toggle with use_aruco:=false. -->
+  <!-- ArUco PLANO en el techo (config original). Solo cuando NO se usa el soporte 3D;
+       con use_soporte:=true lo reemplaza el ArUco 3D del jetauto_soporte. -->
+  <xacro:unless value="$(arg use_soporte)">
   <xacro:if value="$(arg use_aruco)">
     <link name="techo_aruco_link">
@@ -66,3 +71,8 @@
     </joint>
   </xacro:if>
+  </xacro:unless>
+  <!-- Soporte 3D (Legera) + ArUco 3D (ID 4) + MS200 funcional sobre el soporte. -->
+  <xacro:if value="$(arg use_soporte)">
+    <xacro:jetauto_soporte prefix="$(arg prefix)"/>
+  </xacro:if>
 </robot>
