Commit message: Isaac port (Kalman + GridMap), EKF manual y mejoras de sim/mision
isaac/ (nuevo):
- Versiones cinematicas en Isaac: kf_control_isaac, gridmap_isaac y sus
  escenas (scene_agv, scene_gridmap), modelos (rover_model, sensor_models),
  materiales y launch/rviz de visualizacion
- URDFs exportados (jetauto, jetauto_full), textura, env y scripts run_*

ekf_manual/ (nuevo):
- Nodo EKF mecanum manual (ekf_manual_node, ekf_model), launch de
  comparacion, rviz, script run_ekf y README

mi_proyecto_sim:
- Launches nuevos (localizacion_nav_amcl_bridge, navegacion_slam,
  solo_carrito_obstaculos_lidar) y ajustes en bringup/sim/mapeo/simulacion
- Nodos: control_diferencial, control_trayectoria, generador_mapa,
  jetauto_chassis_sim, mision_dron, nav_goal_bridge
- Mision/stitching: stitch_pose (py + cpp nuevo), blend_vote
- Mallas laberinto_real: reemplazo de cajas/conos/cubos/obstaculosFix por
  cajasRecientes; URDF base, world y model.sdf actualizados
- Mallas jetauto extra (jetson decimado, back_shell, aruco) y mapas/arucos

.gitignore:
- Ignora rf2o_laser_odometry/ (trae su propio .git, igual que demo_tello_sim)
- Ignora artefactos regenerables de Isaac (figs/, .ament_overlay/)

File: src/mi_proyecto_sim/urdf/jetauto/jetauto_base.urdf.xacro (robot description, xacro)
@@ -63,5 +63,5 @@
       <visual>
         <origin xyz="0 0 0" rpy="0 0 0"/>
-        <geometry><mesh filename="${mesh_dir}/back_shell_link.stl"/></geometry>
+        <geometry><mesh filename="${mesh_dir}/back_shell_noant.stl"/></geometry>   <!-- sin antenas -->
         <material name="shell_black"><color rgba="0.1 0.1 0.1 1.0"/></material>
       </visual>
